File: board/Comm.sch (KiCad schematic (older format))
At the start: 2 parts, among them J41 WiFi, J42 GPRS

Commit message: Circuit completed, PCB design is next.
Parts:
- J41, J42: footprint (none) -> Pin_Headers:Pin_Header_Straight_2x04
Changed lines of the file:
@@
 EESchema Schematic File Version 2
+LIBS:board-rescue
 LIBS:power
 LIBS:device
@@
 LIBS:leds
 LIBS:L293D
-LIBS:board-cache
 EELAYER 25 0
 EELAYER END
@@
 F 0 "J41" H 3050 1900 50  0000 C CNN
 F 1 "WiFi" H 3050 1400 50  0000 C CNN
-F 2 "" H 3050 450 50  0001 C CNN
+F 2 "Pin_Headers:Pin_Header_Straight_2x04" H 3050 450 50  0001 C CNN
 F 3 "" H 3050 450 50  0001 C CNN
 	1    3050 1650
@@
 F 0 "J42" H 3100 2900 50  0000 C CNN
 F 1 "GPRS" H 3100 2400 50  0000 C CNN
-F 2 "" H 3100 1450 50  0001 C CNN
+F 2 "Pin_Headers:Pin_Header_Straight_2x04" H 3100 1450 50  0001 C CNN
 F 3 "" H 3100 1450 50  0001 C CNN
 	1    3100 2650
