File: board/LCD.sch (KiCad schematic (older format))
At the start: 5 parts, among them Q1 BC547

Commit message: Circuit completed, PCB design is next.
Parts:
- DS1: footprint (none) -> Displays:WC1602A
- Q1: footprint TO_SOT_Packages_THT:TO-92_Molded_Narrow -> TO_SOT_Packages_THT:TO-92_Inline_Narrow_Oval
- R1, R2, R3: footprint (none) -> Resistors_SMD:R_0805
Changed lines of the file:
@@
 EESchema Schematic File Version 2
+LIBS:board-rescue
 LIBS:power
 LIBS:device
@@
 LIBS:leds
 LIBS:L293D
-LIBS:board-cache
 EELAYER 25 0
 EELAYER END
@@
 F 0 "DS1" H 3950 2600 50  0000 C CNN
 F 1 "LCD16X2" H 5450 2600 50  0000 C CNN
-F 2 "" H 4750 2150 50  0001 C CIN
+F 2 "Displays:WC1602A" H 4750 2150 50  0001 C CIN
 F 3 "" H 4750 2200 50  0001 C CNN
 	1    4750 2200
@@
 F 0 "Q1" H 6050 2875 50  0000 L CNN
 F 1 "BC547" H 6050 2800 50  0000 L CNN
-F 2 "TO_SOT_Packages_THT:TO-92_Molded_Narrow" H 6050 2725 50  0001 L CIN
+F 2 "TO_SOT_Packages_THT:TO-92_Inline_Narrow_Oval" H 6050 2725 50  0001 L CIN
 F 3 "" H 5850 2800 50  0001 L CNN
 	1    5850 2800
@@
 F 0 "R2" H 5430 2970 50  0000 L CNN
 F 1 "5k" H 5430 2910 50  0000 L CNN
-F 2 "" H 5400 2950 50  0001 C CNN
+F 2 "Resistors_SMD:R_0805" H 5400 2950 50  0001 C CNN
 F 3 "" H 5400 2950 50  0001 C CNN
 	1    5400 2950
@@
 F 0 "R3" H 5880 3270 50  0000 L CNN
 F 1 "1k" H 5880 3210 50  0000 L CNN
-F 2 "" H 5850 3250 50  0001 C CNN
+F 2 "Resistors_SMD:R_0805" H 5850 3250 50  0001 C CNN
 F 3 "" H 5850 3250 50  0001 C CNN
 	1    5850 3250
@@
 F 0 "R1" V 4230 2870 50  0000 L CNN
 F 1 "1k" H 4230 2810 50  0000 L CNN
-F 2 "" H 4200 2850 50  0001 C CNN
+F 2 "Resistors_SMD:R_0805" H 4200 2850 50  0001 C CNN
 F 3 "" H 4200 2850 50  0001 C CNN
 	1    4200 2850
