File: board/LED_DRIVER5.sch (KiCad schematic (older format))
At the start: 5 parts, among them IC5 L293D, J25 LED_OUT17, J26 LED_OUT18, J27 LED_OUT19, J28 LED_OUT20

Commit message: Circuit completed, PCB design is next.
Parts:
- IC5: footprint (none) -> Housings_DIP:DIP-16_W7.62mm
- J25, J26, J27, J28: footprint (none) -> Connectors_Terminal_Blocks:TerminalBlock_Pheonix_MPT-2.54mm_2pol
Changed lines of the file:
@@
 EESchema Schematic File Version 2
+LIBS:board-rescue
 LIBS:power
 LIBS:device
@@
 LIBS:leds
 LIBS:L293D
-LIBS:board-cache
 EELAYER 25 0
 EELAYER END
@@
 F 0 "IC5" H 5150 4590 50  0000 L BNN
 F 1 "L293D" H 5150 2850 50  0000 L BNN
-F 2 "" H 5550 3750 50  0001 L BNN
+F 2 "Housings_DIP:DIP-16_W7.62mm" H 5550 3750 50  0001 L BNN
 F 3 "STMicroelectronics" H 5550 3750 50  0001 L BNN
 F 4 "Driver%3B 36V%3B Power DIP%3B 600mA Low LevelO/P%3B 1.2A O/P High Level%3B 4 Drivers%3B 7V" H 5550 3750 50  0001 L BNN "Description"
@@
 F 0 "J25" H 2750 3550 50  0000 C TNN
 F 1 "LED_OUT17" V 2600 3300 50  0000 C TNN
-F 2 "" H 2750 3075 50  0001 C CNN
+F 2 "Connectors_Terminal_Blocks:TerminalBlock_Pheonix_MPT-2.54mm_2pol" H 2750 3075 50  0001 C CNN
 F 3 "" H 2725 3300 50  0001 C CNN
 	1    2750 3300
@@
 F 0 "J26" H 2750 4100 50  0000 C TNN
 F 1 "LED_OUT18" V 2600 3850 50  0000 C TNN
-F 2 "" H 2750 3625 50  0001 C CNN
+F 2 "Connectors_Terminal_Blocks:TerminalBlock_Pheonix_MPT-2.54mm_2pol" H 2750 3625 50  0001 C CNN
 F 3 "" H 2725 3850 50  0001 C CNN
 	1    2750 3850
@@
 F 0 "J27" H 2750 4650 50  0000 C TNN
 F 1 "LED_OUT19" V 2600 4400 50  0000 C TNN
-F 2 "" H 2750 4175 50  0001 C CNN
+F 2 "Connectors_Terminal_Blocks:TerminalBlock_Pheonix_MPT-2.54mm_2pol" H 2750 4175 50  0001 C CNN
 F 3 "" H 2725 4400 50  0001 C CNN
 	1    2750 4400
@@
 F 0 "J28" H 2750 5200 50  0000 C TNN
 F 1 "LED_OUT20" V 2600 4950 50  0000 C TNN
-F 2 "" H 2750 4725 50  0001 C CNN
+F 2 "Connectors_Terminal_Blocks:TerminalBlock_Pheonix_MPT-2.54mm_2pol" H 2750 4725 50  0001 C CNN
 F 3 "" H 2725 4950 50  0001 C CNN
 	1    2750 4950
