File: board/RGB_LED_DRIVER.sch (KiCad schematic (older format))
At the start: 4 parts, among them J43 RGB1, J44 RGB2, J45 RGB4, J46 RGB3

Commit message: Circuit completed, PCB design is next.
Parts:
- J43, J44, J45, J46: footprint (none) -> Connectors_Terminal_Blocks:TerminalBlock_Pheonix_MPT-2.54mm_3pol
Changed lines of the file:
@@
 EESchema Schematic File Version 2
+LIBS:board-rescue
 LIBS:power
 LIBS:device
@@
 LIBS:leds
 LIBS:L293D
-LIBS:board-cache
 EELAYER 25 0
 EELAYER END
@@
 F 0 "J43" H 2050 2350 50  0000 C TNN
 F 1 "RGB1" V 1900 2000 50  0000 C TNN
-F 2 "" H 2050 1675 50  0001 C CNN
+F 2 "Connectors_Terminal_Blocks:TerminalBlock_Pheonix_MPT-2.54mm_3pol" H 2050 1675 50  0001 C CNN
 F 3 "" H 2025 2100 50  0001 C CNN
 	1    2050 2000
@@
 F 0 "J44" H 2100 3700 50  0000 C TNN
 F 1 "RGB2" V 1950 3350 50  0000 C TNN
-F 2 "" H 2100 3025 50  0001 C CNN
+F 2 "Connectors_Terminal_Blocks:TerminalBlock_Pheonix_MPT-2.54mm_3pol" H 2100 3025 50  0001 C CNN
 F 3 "" H 2075 3450 50  0001 C CNN
 	1    2100 3350
@@
 F 0 "J45" H 3950 2300 50  0000 C TNN
 F 1 "RGB4" V 3800 1950 50  0000 C TNN
-F 2 "" H 3950 1625 50  0001 C CNN
+F 2 "Connectors_Terminal_Blocks:TerminalBlock_Pheonix_MPT-2.54mm_3pol" H 3950 1625 50  0001 C CNN
 F 3 "" H 3925 2050 50  0001 C CNN
 	1    3950 1950
@@
 F 0 "J46" H 3950 3650 50  0000 C TNN
 F 1 "RGB3" V 3800 3300 50  0000 C TNN
-F 2 "" H 3950 2975 50  0001 C CNN
+F 2 "Connectors_Terminal_Blocks:TerminalBlock_Pheonix_MPT-2.54mm_3pol" H 3950 2975 50  0001 C CNN
 F 3 "" H 3925 3400 50  0001 C CNN
 	1    3950 3300
