File: board/SENSORS.sch (KiCad schematic (older format))
At the start: 47 parts, among them J33 Ain-0, J34 Ain-1, J35 Ain-2, J36 Ain-3, J37 Ain-4, J38 Ain-6, J39 Ain-5, J40 CONN_02X09, U5 10k, U6 10k

Commit message: Circuit completed, PCB design is next.
Parts:
- C17, C18, C19, C20, C21, C22, C23: footprint (none) -> Capacitors_SMD:C_0805
- D10, D11, D12, D13, D7, D8, D9: footprint (none) -> Diodes_SMD:D_1206
- J33, J34, J35, J36, J37, J38, J39: footprint (none) -> Connectors:BARREL_JACK
- J40: footprint (none) -> Pin_Headers:Pin_Header_Straight_2x09
- R11, R12, R13, R14, R15, R16, R17, R18, R19, R20, R21, R22, R23, R24, R25, R26, R27, R28, R29, R30, R31, R32, R33: footprint (none) -> Resistors_SMD:R_0805
- U5, U6: value 10k -> 4n25; symbol 4N25 -> 4N25-RESCUE-board
