File: board/board.sch (KiCad schematic (older format))
At the start: 17 parts, among them J1 BARREL_JACK, U1 LM2596S-5, U2 AMS1117

Commit message: Circuit completed, PCB design is next.
Parts:
- C1, C2: footprint (none) -> Capacitors_THT:CP_Radial_D5.0mm_P2.50mm
- C3, C5: footprint (none) -> Capacitors_THT:CP_Radial_D8.0mm_P3.80mm
- C4: footprint (none) -> Capacitors_SMD:C_0805
- D1, D2: footprint Diodes_THT:D_DO-41_SOD81_Horizontal_RM10 -> Diodes_THT:D_DO-41_SOD81_P7.62mm_Horizontal
- D3: footprint Diodes_THT:D_DO-201AD_Horizontal_RM15 -> Diodes_SMD:D_1206
- J1: footprint (none) -> Connectors:BARREL_JACK
- L1: footprint (none) -> Choke_SMD:Choke_SMD_6.3x6.3_H3
- Pin1, PinLED1, PinRGB1, Pout1, Pout2: footprint (none) -> Connectors_Terminal_Blocks:TerminalBlock_Pheonix_MPT-2.54mm_2pol
- U2: footprint (none) -> TO_SOT_Packages_SMD:SOT-223-3Lead_TabPin2
Changed lines of the file:
@@
 EESchema Schematic File Version 2
+LIBS:board-rescue
 LIBS:power
 LIBS:device
@@
 LIBS:leds
 LIBS:L293D
-LIBS:board-cache
 EELAYER 25 0
 EELAYER END
@@
 F 0 "J1" H 1400 1495 50  0000 C CNN
 F 1 "BARREL_JACK" H 1400 1145 50  0000 C CNN
-F 2 "" H 1400 1300 50  0001 C CNN
+F 2 "Connectors:BARREL_JACK" H 1400 1300 50  0001 C CNN
 F 3 "" H 1400 1300 50  0001 C CNN
 	1    1400 1300
@@
 F 0 "C1" H 2510 1420 50  0000 L CNN
 F 1 "40V, 100uF" H 2510 1270 50  0000 L CNN
-F 2 "" H 2500 1350 50  0001 C CNN
+F 2 "Capacitors_THT:CP_Radial_D5.0mm_P2.50mm" H 2500 1350 50  0001 C CNN
 F 3 "" H 2500 1350 50  0001 C CNN
 	1    2500 1350
@@
 F 0 "D3" H 4300 1550 50  0000 C CNN
 F 1 "1N5822" H 4300 1350 50  0000 C CNN
-F 2 "Diodes_THT:D_DO-201AD_Horizontal_RM15" H 4300 1275 50  0001 C CNN
+F 2 "Diodes_SMD:D_1206" H 4300 1275 50  0001 C CNN
 F 3 "" H 4300 1450 50  0001 C CNN
 	1    4300 1450
@@
 F 0 "L1" V 4450 900 50  0000 C CNN
 F 1 "33uH, 3A" V 4575 900 50  0000 C CNN
-F 2 "" H 4500 900 50  0001 C CNN
+F 2 "Choke_SMD:Choke_SMD_6.3x6.3_H3" H 4500 900 50  0001 C CNN
 F 3 "" H 4500 900 50  0001 C CNN
 	1    4500 900
@@
 F 0 "C2" H 4710 1570 50  0000 L CNN
 F 1 "220uF" H 4710 1420 50  0000 L CNN
-F 2 "" H 4700 1500 50  0001 C CNN
+F 2 "Capacitors_THT:CP_Radial_D5.0mm_P2.50mm" H 4700 1500 50  0001 C CNN
 F 3 "" H 4700 1500 50  0001 C CNN
 	1    4700 1500
@@
 F 0 "C4" H 5510 3820 50  0000 L CNN
 F 1 "22uF" H 5510 3670 50  0000 L CNN
-F 2 "" H 5500 3750 50  0001 C CNN
+F 2 "Capacitors_SMD:C_0805" H 5500 3750 50  0001 C CNN
 F 3 "" H 5500 3750 50  0001 C CNN
 	1    5500 3750
@@
 F 0 "Pin1" H 1450 2800 50  0000 C TNN
 F 1 "Pin" V 1300 2550 50  0000 C TNN
-F 2 "" H 1450 2325 50  0001 C CNN
+F 2 "Connectors_Terminal_Blocks:TerminalBlock_Pheonix_MPT-2.54mm_2pol" H 1450 2325 50  0001 C CNN
 F 3 "" H 1425 2550 50  0001 C CNN
 	1    1450 2550
@@
 F 0 "Pout1" H 1450 3500 50  0000 C TNN
 F 1 "5V" V 1300 3250 50  0000 C TNN
-F 2 "" H 1450 3025 50  0001 C CNN
+F 2 "Connectors_Terminal_Blocks:TerminalBlock_Pheonix_MPT-2.54mm_2pol" H 1450 3025 50  0001 C CNN
 F 3 "" H 1425 3250 50  0001 C CNN
 	1    1450 3250
@@
 F 0 "C3" H 5075 1350 50  0000 L CNN
 F 1 "CP15V, 1000uF" H 5075 1150 50  0000 L CNN
-F 2 "" H 5050 1250 50  0001 C CNN
+F 2 "Capacitors_THT:CP_Radial_D8.0mm_P3.80mm" H 5050 1250 50  0001 C CNN
 F 3 "" H 5050 1250 50  0001 C CNN
 	1    5050 1250
@@
 F 0 "C5" H 5875 1350 50  0000 L CNN
 F 1 "5V, 1000uF" H 5875 1150 50  0000 L CNN
-F 2 "" H 5850 1250 50  0001 C CNN
+F 2 "Capacitors_THT:CP_Radial_D8.0mm_P3.80mm" H 5850 1250 50  0001 C CNN
 F 3 "" H 5850 1250 50  0001 C CNN
 	1    5850 1250
@@
 F 0 "PinRGB1" H 1450 4350 50  0000 C TNN
 F 1 "RGB Vcc" V 1300 4100 50  0000 C TNN
-F 2 "" H 1450 3875 50  0001 C CNN
+F 2 "Connectors_Terminal_Blocks:TerminalBlock_Pheonix_MPT-2.54mm_2pol" H 1450 3875 50  0001 C CNN
 F 3 "" H 1425 4100 50  0001 C CNN
 	1    1450 4100
@@
 F 0 "PinLED1" H 2800 3150 50  0000 C TNN
 F 1 "LED Vcc" V 2650 2900 50  0000 C TNN
-F 2 "" H 2800 2675 50  0001 C CNN
+F 2 "Connectors_Terminal_Blocks:TerminalBlock_Pheonix_MPT-2.54mm_2pol" H 2800 2675 50  0001 C CNN
 F 3 "" H 2775 2900 50  0001 C CNN
 	1    2800 2900
@@
 F 0 "D2" H 1950 1300 50  0000 C CNN
 F 1 "1N4007" H 1950 1100 50  0000 C CNN
-F 2 "Diodes_THT:D_DO-41_SOD81_Horizontal_RM10" H 1950 1025 50  0001 C CNN
+F 2 "Diodes_THT:D_DO-41_SOD81_P7.62mm_Horizontal" H 1950 1025 50  0001 C CNN
 F 3 "" H 1950 1200 50  0001 C CNN
 	1    1950 1200
@@
 F 0 "D1" H 1950 1000 50  0000 C CNN
 F 1 "1N4007" H 1950 800 50  0000 C CNN
-F 2 "Diodes_THT:D_DO-41_SOD81_Horizontal_RM10" H 1950 725 50  0001 C CNN
+F 2 "Diodes_THT:D_DO-41_SOD81_P7.62mm_Horizontal" H 1950 725 50  0001 C CNN
 F 3 "" H 1950 900 50  0001 C CNN
 	1    1950 900
@@
 F 0 "Pout2" H 2800 4250 50  0000 C TNN
 F 1 "Vcc Out" V 2650 4000 50  0000 C TNN
-F 2 "" H 2800 3775 50  0001 C CNN
+F 2 "Connectors_Terminal_Blocks:TerminalBlock_Pheonix_MPT-2.54mm_2pol" H 2800 3775 50  0001 C CNN
 F 3 "" H 2775 4000 50  0001 C CNN
 	1    2800 4000
@@
 F 0 "U2" H 5000 3850 50  0000 C CNN
 F 1 "AMS1117" H 5050 3300 50  0000 L CNN
-F 2 "" H 5000 3550 50  0001 C CNN
+F 2 "TO_SOT_Packages_SMD:SOT-223-3Lead_TabPin2" H 5000 3550 50  0001 C CNN
 F 3 "" H 5000 3550 50  0001 C CNN
 	1    5000 3550
