File: board/controller.sch (KiCad schematic (older format))
At the start: 34 parts, among them J2 ICSP, J3 Port J, J4 Port L, J5 Port H, J6 Port C, J7 USB_B, J8 Comm, Q2 BC547, SW1 reset, U3 ATMEGA1280-16AU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

Commit message: Circuit completed, PCB design is next.
Parts:
- C10, C11, C12, C13, C14, C15, C16, C6, C7, C8, C9: footprint (none) -> Capacitors_SMD:C_0805
- D4, D5, D6: footprint (none) -> LEDs:LED_0805
- F1: footprint (none) -> Resistors_SMD:R_1206
- J2: footprint (none) -> Socket_Strips:Socket_Strip_Straight_2x03
- J3: footprint (none) -> Pin_Headers:Pin_Header_Straight_1x05
- J4, J6: footprint (none) -> Pin_Headers:Pin_Header_Straight_1x08
- J5, J8: footprint (none) -> Pin_Headers:Pin_Header_Straight_1x02
- J7: footprint (none) -> Connectors:USB_B
- Q2: footprint TO_SOT_Packages_THT:TO-92_Molded_Narrow -> TO_SOT_Packages_THT:TO-92_Inline_Narrow_Oval
- R10, R4, R5, R6, R7, R8, R9: footprint (none) -> Resistors_SMD:R_0805
- SW1: footprint (none) -> Buttons_Switches_SMD:SW_SPST_B3S-1000
- U3: footprint (none) -> Housings_QFP:TQFP-100_14x14mm_Pitch0.5mm
- U4: footprint (none) -> Housings_SSOP:SSOP-28_5.3x10.2mm_Pitch0.65mm
- Y1: footprint (none) -> Crystals:Crystal_HC49-SD_SMD
Changed lines of the file:
@@
 EESchema Schematic File Version 2
+LIBS:board-rescue
 LIBS:power
 LIBS:device
@@
 LIBS:leds
 LIBS:L293D
-LIBS:board-cache
 EELAYER 25 0
 EELAYER END
@@
 F 0 "U3" H 3850 6950 50  0000 L BNN
 F 1 "ATMEGA1280-16AU" H 5700 1300 50  0000 L BNN
-F 2 "" H 5000 4150 50  0001 C CIN
+F 2 "Housings_QFP:TQFP-100_14x14mm_Pitch0.5mm" H 5000 4150 50  0001 C CIN
 F 3 "" H 5000 4150 50  0001 C CNN
 	1    5000 4150
@@
 F 0 "C10" H 5410 1120 50  0000 L CNN
 F 1 "100nF" H 5410 970 50  0000 L CNN
-F 2 "" H 5400 1050 50  0001 C CNN
+F 2 "Capacitors_SMD:C_0805" H 5400 1050 50  0001 C CNN
 F 3 "" H 5400 1050 50  0001 C CNN
 	1    5400 1050
@@
 F 0 "C11" H 5660 1120 50  0000 L CNN
 F 1 "100nF" H 5660 970 50  0000 L CNN
-F 2 "" H 5650 1050 50  0001 C CNN
+F 2 "Capacitors_SMD:C_0805" H 5650 1050 50  0001 C CNN
 F 3 "" H 5650 1050 50  0001 C CNN
 	1    5650 1050
@@
 F 0 "C12" H 5910 1120 50  0000 L CNN
 F 1 "100nF" H 5910 970 50  0000 L CNN
-F 2 "" H 5900 1050 50  0001 C CNN
+F 2 "Capacitors_SMD:C_0805" H 5900 1050 50  0001 C CNN
 F 3 "" H 5900 1050 50  0001 C CNN
 	1    5900 1050
@@
 F 0 "Y1" H 3500 2100 50  0000 C CNN
 F 1 "16Mhz" H 3500 1900 50  0000 C CNN
-F 2 "" H 3500 2000 50  0001 C CNN
+F 2 "Crystals:Crystal_HC49-SD_SMD" H 3500 2000 50  0001 C CNN
 F 3 "" H 3500 2000 50  0001 C CNN
 	1    3500 2000
@@
 F 0 "C6" H 3160 1920 50  0000 L CNN
 F 1 "22pF" H 3160 1770 50  0000 L CNN
-F 2 "" H 3150 1850 50  0001 C CNN
+F 2 "Capacitors_SMD:C_0805" H 3150 1850 50  0001 C CNN
 F 3 "" H 3150 1850 50  0001 C CNN
 	1    3150 1850
@@
 F 0 "C7" H 3160 2220 50  0000 L CNN
 F 1 "22p" H 3160 2070 50  0000 L CNN
-F 2 "" H 3150 2150 50  0001 C CNN
+F 2 "Capacitors_SMD:C_0805" H 3150 2150 50  0001 C CNN
 F 3 "" H 3150 2150 50  0001 C CNN
 	1    3150 2150
@@
 F 0 "C9" H 3710 7070 50  0000 L CNN
 F 1 "100n" H 3710 6920 50  0000 L CNN
-F 2 "" H 3700 7000 50  0001 C CNN
+F 2 "Capacitors_SMD:C_0805" H 3700 7000 50  0001 C CNN
 F 3 "" H 3700 7000 50  0001 C CNN
 	1    3700 7000
@@
 F 0 "C8" H 3360 1620 50  0000 L CNN
 F 1 "100n" H 3360 1470 50  0000 L CNN
-F 2 "" H 3350 1550 50  0001 C CNN
+F 2 "Capacitors_SMD:C_0805" H 3350 1550 50  0001 C CNN
 F 3 "" H 3350 1550 50  0001 C CNN
 	1    3350 1550
@@
 F 0 "R4" H 3530 1270 50  0000 L CNN
 F 1 "10k" H 3530 1210 50  0000 L CNN
-F 2 "" H 3500 1250 50  0001 C CNN
+F 2 "Resistors_SMD:R_0805" H 3500 1250 50  0001 C CNN
 F 3 "" H 3500 1250 50  0001 C CNN
 	1    3500 1250
@@
 F 0 "SW1" H 3150 1200 50  0000 L CNN
 F 1 "reset" H 3100 1040 50  0000 C CNN
-F 2 "" H 3100 1300 50  0001 C CNN
+F 2 "Buttons_Switches_SMD:SW_SPST_B3S-1000" H 3100 1300 50  0001 C CNN
 F 3 "" H 3100 1300 50  0001 C CNN
 	1    3100 1100
@@
 F 0 "U4" H 8500 3700 50  0000 L CNN
 F 1 "FT232RL" H 9550 3700 50  0000 L CNN
-F 2 "" H 9150 2800 50  0001 C CNN
+F 2 "Housings_SSOP:SSOP-28_5.3x10.2mm_Pitch0.65mm" H 9150 2800 50  0001 C CNN
 F 3 "" H 9150 2800 50  0001 C CNN
 	1    9150 2800
@@
 F 0 "D5" H 10100 3050 50  0000 C CNN
 F 1 "Rx" H 10100 2850 50  0000 C CNN
-F 2 "" H 10100 2950 50  0001 C CNN
+F 2 "LEDs:LED_0805" H 10100 2950 50  0001 C CNN
 F 3 "" H 10100 2950 50  0001 C CNN
 	1    10100 2950
@@
 F 0 "D6" H 10400 3050 50  0000 C CNN
 F 1 "TX" H 10400 2850 50  0000 C CNN
-F 2 "" H 10400 2950 50  0001 C CNN
+F 2 "LEDs:LED_0805" H 10400 2950 50  0001 C CNN
 F 3 "" H 10400 2950 50  0001 C CNN
 	1    10400 2950
@@
 F 0 "R7" H 10130 2670 50  0000 L CNN
 F 1 "1k" H 10130 2610 50  0000 L CNN
-F 2 "" H 10100 2650 50  0001 C CNN
+F 2 "Resistors_SMD:R_0805" H 10100 2650 50  0001 C CNN
 F 3 "" H 10100 2650 50  0001 C CNN
 	1    10100 2650
@@
 F 0 "R9" H 10430 2670 50  0000 L CNN
 F 1 "1k" H 10430 2610 50  0000 L CNN
-F 2 "" H 10400 2650 50  0001 C CNN
+F 2 "Resistors_SMD:R_0805" H 10400 2650 50  0001 C CNN
 F 3 "" H 10400 2650 50  0001 C CNN
 	1    10400 2650
@@
 F 0 "C16" H 10710 2520 50  0000 L CNN
 F 1 "100n" V 10710 2370 50  0000 L CNN
-F 2 "" H 10700 2450 50  0001 C CNN
+F 2 "Capacitors_SMD:C_0805" H 10700 2450 50  0001 C CNN
 F 3 "" H 10700 2450 50  0001 C CNN
 	1    10700 2450
@@
 F 0 "R10" H 10480 2120 50  0000 L CNN
 F 1 "1k" H 10480 2060 50  0000 L CNN
-F 2 "" H 10450 2100 50  0001 C CNN
+F 2 "Resistors_SMD:R_0805" H 10450 2100 50  0001 C CNN
 F 3 "" H 10450 2100 50  0001 C CNN
 	1    10450 2100
@@
 F 0 "R8" H 10180 2220 50  0000 L CNN
 F 1 "1k" H 10180 2160 50  0000 L CNN
-F 2 "" H 10150 2200 50  0001 C CNN
+F 2 "Resistors_SMD:R_0805" H 10150 2200 50  0001 C CNN
 F 3 "" H 10150 2200 50  0001 C CNN
 	1    10150 2200
@@
 F 0 "C13" H 8010 3020 50  0000 L CNN
 F 1 "100n" H 8010 2870 50  0000 L CNN
-F 2 "" H 8000 2950 50  0001 C CNN
+F 2 "Capacitors_SMD:C_0805" H 8000 2950 50  0001 C CNN
 F 3 "" H 8000 2950 50  0001 C CNN
 	1    8000 2950
@@
 F 0 "J7" H 7350 2500 50  0000 L CNN
 F 1 "USB_B" H 7350 2400 50  0000 L CNN
-F 2 "" H 7700 2000 50  0001 C CNN
+F 2 "Connectors:USB_B" H 7700 2000 50  0001 C CNN
 F 3 "" H 7700 2000 50  0001 C CNN
 	1    7550 2050
@@
 F 0 "C15" H 8260 1770 50  0000 L CNN
 F 1 "100n" H 8260 1620 50  0000 L CNN
-F 2 "" H 8250 1700 50  0001 C CNN
+F 2 "Capacitors_SMD:C_0805" H 8250 1700 50  0001 C CNN
 F 3 "" H 8250 1700 50  0001 C CNN
 	1    8250 1700
@@
 F 0 "C14" H 8260 1520 50  0000 L CNN
 F 1 "100n" H 8260 1370 50  0000 L CNN
-F 2 "" H 8250 1450 50  0001 C CNN
+F 2 "Capacitors_SMD:C_0805" H 8250 1450 50  0001 C CNN
 F 3 "" H 8250 1450 50  0001 C CNN
 	1    8250 1450
@@
 F 0 "F1" V 7775 1500 50  0000 C CNN
 F 1 "500mA" V 7925 1500 50  0000 C CNN
-F 2 "" H 7900 1300 50  0001 L CNN
+F 2 "Resistors_SMD:R_1206" H 7900 1300 50  0001 L CNN
 F 3 "" H 7850 1500 50  0001 C CNN
 	1    7850 1500
@@
 F 0 "D4" H 7450 3500 50  0000 C CNN
 F 1 "LED_ALT" H 7450 3300 50  0000 C CNN
-F 2 "" H 7450 3400 50  0001 C CNN
+F 2 "LEDs:LED_0805" H 7450 3400 50  0001 C CNN
 F 3 "" H 7450 3400 50  0001 C CNN
 	1    7450 3400
@@
 F 0 "R5" H 7080 3420 50  0000 L CNN
 F 1 "1k" H 7080 3360 50  0000 L CNN
-F 2 "" H 7050 3400 50  0001 C CNN
+F 2 "Resistors_SMD:R_0805" H 7050 3400 50  0001 C CNN
 F 3 "" H 7050 3400 50  0001 C CNN
 	1    7050 3400
@@
 F 0 "Q2" H 9350 4575 50  0000 L CNN
 F 1 "BC547" H 9350 4500 50  0000 L CNN
-F 2 "TO_SOT_Packages_THT:TO-92_Molded_Narrow" H 9350 4425 50  0001 L CIN
+F 2 "TO_SOT_Packages_THT:TO-92_Inline_Narrow_Oval" H 9350 4425 50  0001 L CIN
 F 3 "" H 9150 4500 50  0001 L CNN
 	1    9150 4500
@@
 F 0 "R6" H 9280 4920 50  0000 L CNN
 F 1 "5k" H 9280 4860 50  0000 L CNN
-F 2 "" H 9250 4900 50  0001 C CNN
+F 2 "Resistors_SMD:R_0805" H 9250 4900 50  0001 C CNN
 F 3 "" H 9250 4900 50  0001 C CNN
 	1    9250 4900
@@
 F 0 "J2" H 1450 1250 50  0000 C CNN
 F 1 "ICSP" H 1450 850 50  0000 C CNN
-F 2 "" H 1450 -150 50  0001 C CNN
+F 2 "Socket_Strips:Socket_Strip_Straight_2x03" H 1450 -150 50  0001 C CNN
 F 3 "" H 1450 -150 50  0001 C CNN
 	1    1450 1050
@@
 F 0 "J4" H 2850 3250 50  0000 C CNN
 F 1 "Port L" V 2950 2800 50  0000 C CNN
-F 2 "" H 2850 2800 50  0001 C CNN
+F 2 "Pin_Headers:Pin_Header_Straight_1x08" H 2850 2800 50  0001 C CNN
 F 3 "" H 2850 2800 50  0001 C CNN
 	1    2850 2800
@@
 F 0 "J3" H 2800 5050 50  0000 C CNN
 F 1 "Port J" V 2900 4750 50  0000 C CNN
-F 2 "" H 2800 4750 50  0001 C CNN
+F 2 "Pin_Headers:Pin_Header_Straight_1x05" H 2800 4750 50  0001 C CNN
 F 3 "" H 2800 4750 50  0001 C CNN
 	1    2800 4750
@@
 F 0 "J5" H 2850 5950 50  0000 C CNN
 F 1 "Port H" V 2950 5800 50  0000 C CNN
-F 2 "" H 2850 5800 50  0001 C CNN
+F 2 "Pin_Headers:Pin_Header_Straight_1x02" H 2850 5800 50  0001 C CNN
 F 3 "" H 2850 5800 50  0001 C CNN
 	1    2850 5800
@@
 F 0 "J6" H 7200 3250 50  0000 C CNN
 F 1 "Port C" V 7300 2800 50  0000 C CNN
-F 2 "" H 7200 2800 50  0001 C CNN
+F 2 "Pin_Headers:Pin_Header_Straight_1x08" H 7200 2800 50  0001 C CNN
 F 3 "" H 7200 2800 50  0001 C CNN
 	1    7200 2800
@@
 F 0 "J8" H 7600 4400 50  0000 C CNN
 F 1 "Comm" V 7700 4250 50  0000 C CNN
-F 2 "" H 7600 4250 50  0001 C CNN
+F 2 "Pin_Headers:Pin_Header_Straight_1x02" H 7600 4250 50  0001 C CNN
 F 3 "" H 7600 4250 50  0001 C CNN
 	1    7600 4250
